Commit message: Update Docker configuration for noVNC display resolution and modify URDF file paths for docky robot. Remove obsolete docky_gz.urdf and docky_gz.urdf.xacro files, and add support for .xacro files in setup.py.

File: main_ws/description/docky/urdf/docky.urdf (robot description, URDF)
Before this commit: robot docky, 2 links, 1 joints
Links:
- link Hip: geometry collision box size=5.52036 2.47975 4.01113; visual mesh filename=package://description/docky/meshes/stl/Body.stl scale=0.49027 0.71329 0.27273
- link Root: geometry collision box size=2.22490 3.62134 1.40620; visual mesh filename=package://description/docky/meshes/stl/Feet.stl scale=1.00000 0.42205 0.13092
